File: power.kicad_sch (KiCad schematic)
At the start: 5 parts, among them U3 TCR2EE27, U4 MIC5365-3.0YD5

Commit message: Assign Footprints
Parts:
- C15: renamed from C13; footprint (none) -> Capacitor_SMD:C_0603_1608Metric_Pad1.08x0.95mm_HandSolder
- C16: renamed from C8; footprint (none) -> Capacitor_SMD:C_0603_1608Metric_Pad1.08x0.95mm_HandSolder
- C17: renamed from C16; footprint (none) -> Capacitor_SMD:C_0603_1608Metric_Pad1.08x0.95mm_HandSolder
Changed lines of the file:
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@@
 		(dnp no)
 		(fields_autoplaced yes)
-		(property "Reference" "C8"
+		(property "Reference" "C16"
 			(at 170.18 110.4899 0)
 			(effects
@@
 			)
 		)
-		(property "Footprint" ""
+		(property "Footprint" "Capacitor_SMD:C_0603_1608Metric_Pad1.08x0.95mm_HandSolder"
 			(at 167.3352 115.57 0)
 			(effects
@@
 			(project "usb_microphone"
 				(path "/dc202712-23ff-46da-8ec2-2a828c683a4d/d0b66dcc-b67d-4274-be45-69ac5f31ce8f"
-					(reference "C8")
+					(reference "C16")
 					(unit 1)
 				)
@@
 		(dnp no)
 		(fields_autoplaced yes)
-		(property "Reference" "#PWR04"
+		(property "Reference" "#PWR018"
 			(at 172.72 81.28 0)
 			(effects
@@
 			(project "usb_microphone"
 				(path "/dc202712-23ff-46da-8ec2-2a828c683a4d/d0b66dcc-b67d-4274-be45-69ac5f31ce8f"
-					(reference "#PWR04")
+					(reference "#PWR018")
 					(unit 1)
 				)
@@
 		(dnp no)
 		(fields_autoplaced yes)
-		(property "Reference" "C16"
+		(property "Reference" "C17"
 			(at 171.45 80.0099 0)
 			(effects
@@
 			)
 		)
-		(property "Footprint" ""
+		(property "Footprint" "Capacitor_SMD:C_0603_1608Metric_Pad1.08x0.95mm_HandSolder"
 			(at 168.6052 85.09 0)
 			(effects
@@
 			(project "usb_microphone"
 				(path "/dc202712-23ff-46da-8ec2-2a828c683a4d/d0b66dcc-b67d-4274-be45-69ac5f31ce8f"
-					(reference "C16")
+					(reference "C17")
 					(unit 1)
 				)
@@
 		(dnp no)
 		(fields_autoplaced yes)
-		(property "Reference" "#PWR09"
+		(property "Reference" "#PWR016"
 			(at 152.4 93.98 0)
 			(effects
@@
 			(project "usb_microphone"
 				(path "/dc202712-23ff-46da-8ec2-2a828c683a4d/d0b66dcc-b67d-4274-be45-69ac5f31ce8f"
-					(reference "#PWR09")
+					(reference "#PWR016")
 					(unit 1)
 				)
@@
 		(dnp no)
 		(fields_autoplaced yes)
-		(property "Reference" "#PWR021"
+		(property "Reference" "#PWR017"
 			(at 152.4 124.46 0)
 			(effects
@@
 			(project "usb_microphone"
 				(path "/dc202712-23ff-46da-8ec2-2a828c683a4d/d0b66dcc-b67d-4274-be45-69ac5f31ce8f"
-					(reference "#PWR021")
+					(reference "#PWR017")
 					(unit 1)
 				)
@@
 		(on_board yes)
 		(dnp no)
-		(property "Reference" "C13"
+		(property "Reference" "C15"
 			(at 127 80.0099 0)
 			(effects
@@
 			)
 		)
-		(property "Footprint" ""
+		(property "Footprint" "Capacitor_SMD:C_0603_1608Metric_Pad1.08x0.95mm_HandSolder"
 			(at 124.1552 85.09 0)
 			(effects
@@
 			(project "usb_microphone"
 				(path "/dc202712-23ff-46da-8ec2-2a828c683a4d/d0b66dcc-b67d-4274-be45-69ac5f31ce8f"
-					(reference "C13")
+					(reference "C15")
 					(unit 1)
 				)
@@
 		(dnp no)
 		(fields_autoplaced yes)
-		(property "Reference" "#PWR020"
+		(property "Reference" "#PWR015"
 			(at 138.43 111.76 0)
 			(effects
@@
 			(project "usb_microphone"
 				(path "/dc202712-23ff-46da-8ec2-2a828c683a4d/d0b66dcc-b67d-4274-be45-69ac5f31ce8f"
-					(reference "#PWR020")
+					(reference "#PWR015")
 					(unit 1)
 				)
@@
 		(dnp no)
 		(fields_autoplaced yes)
-		(property "Reference" "#PWR01"
+		(property "Reference" "#PWR014"
 			(at 123.19 81.28 0)
 			(effects
@@
 			(project ""
 				(path "/dc202712-23ff-46da-8ec2-2a828c683a4d/d0b66dcc-b67d-4274-be45-69ac5f31ce8f"
-					(reference "#PWR01")
-					(unit 1)
-				)
+					(reference "#PWR014")
+					(unit 1)
+				)
