File: connectors.kicad_sch (KiCad schematic)
At the start: 3 parts, among them J2 IN_R connector, J3 MIC connector, P1 USB_C_Plug_USB2.0

Commit message: Assign Footprints
Parts:
- J3: renamed from J2; footprint (none) -> Connector_PinHeader_1.27mm:PinHeader_1x03_P1.27mm_Vertical
- J4: renamed from J3; footprint (none) -> Connector_PinHeader_2.54mm:PinHeader_1x02_P2.54mm_Vertical
- P1: footprint (none) -> Connector_USB:USB_C_Receptacle_GCT_USB4135-GF-A_6P_TopMnt_Horizontal
Connections:
- net GND: now also P1.S1 (SHIELD)
- no-connect marks 3 -> 2
Changed lines of the file:
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@@
 		(company "Vladyslav Kukharchuk <vladyslavziuziun@gmail.com>")
 	)
-	(no_connect
-		(at 137.16 78.74)
+	(junction
+		(at 144.78 78.74)
+		(diameter 0)
+		(color 0 0 0 0)
 	)
 	(no_connect
@@
 		(pts
 			(xy 138.43 101.6) (xy 146.05 101.6)
+		)
+		(stroke
+			(width 0)
+			(type default)
+		)
+	)
+	(wire
+		(pts
+			(xy 137.16 78.74) (xy 144.78 78.74)
 		)
 		(stroke
@@
 		(on_board yes)
 		(dnp no)
-		(property "Reference" "J3"
+		(property "Reference" "J4"
 			(at 155.448 118.11 0)
 			(effects
@@
 			)
 		)
-		(property "Footprint" ""
+		(property "Footprint" "Connector_PinHeader_2.54mm:PinHeader_1x02_P2.54mm_Vertical"
 			(at 151.13 120.65 0)
 			(effects
@@
 			(project "usb_microphone"
 				(path "/dc202712-23ff-46da-8ec2-2a828c683a4d/3b6bfc3a-3ecd-4bf7-a684-d469f732a0b7"
-					(reference "J3")
+					(reference "J4")
 					(unit 1)
 				)
@@
 		(dnp no)
 		(fields_autoplaced yes)
-		(property "Reference" "J2"
+		(property "Reference" "J3"
 			(at 153.67 100.3299 0)
 			(effects
@@
 			)
 		)
-		(property "Footprint" ""
+		(property "Footprint" "Connector_PinHeader_1.27mm:PinHeader_1x03_P1.27mm_Vertical"
 			(at 151.13 101.6 0)
 			(effects
@@
 			(project ""
 				(path "/dc202712-23ff-46da-8ec2-2a828c683a4d/3b6bfc3a-3ecd-4bf7-a684-d469f732a0b7"
-					(reference "J2")
+					(reference "J3")
 					(unit 1)
 				)
@@
 		(dnp no)
 		(fields_autoplaced yes)
-		(property "Reference" "#PWR022"
+		(property "Reference" "#PWR023"
 			(at 160.02 44.45 0)
 			(effects
@@
 			(project ""
 				(path "/dc202712-23ff-46da-8ec2-2a828c683a4d/3b6bfc3a-3ecd-4bf7-a684-d469f732a0b7"
-					(reference "#PWR022")
+					(reference "#PWR023")
 					(unit 1)
 				)
@@
 		(dnp no)
 		(fields_autoplaced yes)
-		(property "Reference" "#PWR07"
+		(property "Reference" "#PWR022"
 			(at 146.05 127 0)
 			(effects
@@
 			(project "usb_microphone"
 				(path "/dc202712-23ff-46da-8ec2-2a828c683a4d/3b6bfc3a-3ecd-4bf7-a684-d469f732a0b7"
-					(reference "#PWR07")
+					(reference "#PWR022")
 					(unit 1)
 				)
@@
 		(dnp no)
 		(fields_autoplaced yes)
-		(property "Reference" "#PWR023"
+		(property "Reference" "#PWR021"
 			(at 144.78 85.09 0)
 			(effects
@@
 			(project ""
 				(path "/dc202712-23ff-46da-8ec2-2a828c683a4d/3b6bfc3a-3ecd-4bf7-a684-d469f732a0b7"
-					(reference "#PWR023")
+					(reference "#PWR021")
 					(unit 1)
 				)
@@
 		(dnp no)
 		(fields_autoplaced yes)
-		(property "Reference" "#PWR011"
+		(property "Reference" "#PWR020"
 			(at 138.43 107.95 0)
 			(effects
@@
 			(project ""
 				(path "/dc202712-23ff-46da-8ec2-2a828c683a4d/3b6bfc3a-3ecd-4bf7-a684-d469f732a0b7"
-					(reference "#PWR011")
+					(reference "#PWR020")
 					(unit 1)
 				)
@@
 			)
 		)
-		(property "Footprint" ""
+		(property "Footprint" "Connector_USB:USB_C_Receptacle_GCT_USB4135-GF-A_6P_TopMnt_Horizontal"
 			(at 148.59 55.88 0)
 			(effects
@@
 		(dnp no)
 		(fields_autoplaced yes)
-		(property "Reference" "#PWR010"
+		(property "Reference" "#PWR019"
 			(at 138.43 102.87 0)
 			(effects
@@
 			(project ""
 				(path "/dc202712-23ff-46da-8ec2-2a828c683a4d/3b6bfc3a-3ecd-4bf7-a684-d469f732a0b7"
-					(reference "#PWR010")
-					(unit 1)
-				)
+					(reference "#PWR019")
+					(unit 1)
+				)

Commit message: USB replacement and footprint update
Parts:
- removed P1: USB_C_Plug_USB2.0, Connector_USB:USB_C_Receptacle_GCT_USB4135-GF-A_6P_TopMnt_Horizontal, symbol Connector:USB_C_Plug_USB2.0
- added J3: USB_C_Receptacle_USB2.0_16P, Connector_USB:USB_C_Receptacle_GCT_USB4105-xx-A_16P_TopMnt_Horizontal, symbol Connector:USB_C_Receptacle_USB2.0_16P
- renumbered J3 to J4, J4 to J5
Connections:
- net D +: now also J3.A6 (D+)
- net D -: now also J3.A7 (D-)
- net GND: now also J3.A1 (GND), J3.A12 (GND), J3.B1 (GND), J3.B12 (GND), J3.S1 (SHIELD)
- net VBUS: now also J3.A4 (VBUS), J3.A9 (VBUS), J3.B4 (VBUS), J3.B9 (VBUS)
- no-connect marks 2 -> 6
Other:
- moved on the sheet: J4, J5
