File: codec.kicad_sch (KiCad schematic)
At the start: 16 parts, among them U1 PCM2906CDBR, Y1 Crystal

Commit message: Assign Footprints
Parts:
- C10, C11, C12, C9: footprint (none) -> Capacitor_SMD:C_0603_1608Metric_Pad1.08x0.95mm_HandSolder
- C13: renamed from C14; footprint (none) -> Capacitor_SMD:C_0603_1608Metric_Pad1.08x0.95mm_HandSolder
- C14: renamed from C15; footprint (none) -> Capacitor_SMD:C_0603_1608Metric_Pad1.08x0.95mm_HandSolder
- C6: renamed from C1; footprint (none) -> Capacitor_SMD:C_0603_1608Metric_Pad1.08x0.95mm_HandSolder
- C7: renamed from C3; footprint (none) -> Capacitor_SMD:C_0603_1608Metric_Pad1.08x0.95mm_HandSolder
- C8: renamed from C5; footprint (none) -> Capacitor_SMD:C_0603_1608Metric_Pad1.08x0.95mm_HandSolder
- R4: renamed from R6; footprint (none) -> Resistor_SMD:R_0603_1608Metric_Pad0.98x0.95mm_HandSolder
- R5: footprint (none) -> Resistor_SMD:R_0603_1608Metric_Pad0.98x0.95mm_HandSolder
- R6: renamed from R4; footprint (none) -> Resistor_SMD:R_0603_1608Metric_Pad0.98x0.95mm_HandSolder
- R7: renamed from R9; footprint (none) -> Resistor_SMD:R_0603_1608Metric_Pad0.98x0.95mm_HandSolder
- R8: renamed from R10; footprint (none) -> Resistor_SMD:R_0603_1608Metric_Pad0.98x0.95mm_HandSolder
- U2: renamed from U1; footprint DB28_TEX -> Package_SO:SSOP-28_5.3x10.2mm_P0.65mm
- Y1: value Crystal -> 12MHz; footprint (none) -> Crystal:Crystal_HC49-4H_Vertical
Changed lines of the file:
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@@
 		(on_board yes)
 		(dnp no)
-		(property "Reference" "C14"
+		(property "Reference" "C13"
 			(at 204.47 91.186 90)
 			(effects
@@
 			)
 		)
-		(property "Footprint" ""
+		(property "Footprint" "Capacitor_SMD:C_0603_1608Metric_Pad1.08x0.95mm_HandSolder"
 			(at 208.28 96.8248 0)
 			(effects
@@
 			(project "usb_microphone"
 				(path "/dc202712-23ff-46da-8ec2-2a828c683a4d/8b5991ae-ddae-4cba-9bee-b5c93b934b0b"
-					(reference "C14")
+					(reference "C13")
 					(unit 1)
 				)
@@
 		(on_board yes)
 		(dnp no)
-		(property "Reference" "R4"
+		(property "Reference" "R6"
 			(at 111.506 77.978 90)
 			(effects
@@
 			)
 		)
-		(property "Footprint" ""
+		(property "Footprint" "Resistor_SMD:R_0603_1608Metric_Pad0.98x0.95mm_HandSolder"
 			(at 110.49 80.772 90)
 			(effects
@@
 			(project "usb_microphone"
 				(path "/dc202712-23ff-46da-8ec2-2a828c683a4d/8b5991ae-ddae-4cba-9bee-b5c93b934b0b"
-					(reference "R4")
+					(reference "R6")
 					(unit 1)
 				)
@@
 		(on_board yes)
 		(dnp no)
-		(property "Reference" "R6"
+		(property "Reference" "R4"
 			(at 84.836 83.058 90)
 			(effects
@@
 			)
 		)
-		(property "Footprint" ""
+		(property "Footprint" "Resistor_SMD:R_0603_1608Metric_Pad0.98x0.95mm_HandSolder"
 			(at 83.82 85.852 90)
 			(effects
@@
 			(project "usb_microphone"
 				(path "/dc202712-23ff-46da-8ec2-2a828c683a4d/8b5991ae-ddae-4cba-9bee-b5c93b934b0b"
-					(reference "R6")
+					(reference "R4")
 					(unit 1)
 				)
@@
 		(on_board yes)
 		(dnp no)
-		(property "Reference" "#PWR018"
+		(property "Reference" "#PWR07"
 			(at 95.25 109.22 0)
 			(effects
@@
 			(project ""
 				(path "/dc202712-23ff-46da-8ec2-2a828c683a4d/8b5991ae-ddae-4cba-9bee-b5c93b934b0b"
-					(reference "#PWR018")
+					(reference "#PWR07")
 					(unit 1)
 				)
@@
 		(on_board yes)
 		(dnp no)
-		(property "Reference" "#PWR012"
+		(property "Reference" "#PWR08"
 			(at 105.41 96.52 0)
 			(effects
@@
 			(project "usb_microphone"
 				(path "/dc202712-23ff-46da-8ec2-2a828c683a4d/8b5991ae-ddae-4cba-9bee-b5c93b934b0b"
-					(reference "#PWR012")
+					(reference "#PWR08")
 					(unit 1)
 				)
@@
 		(on_board yes)
 		(dnp no)
-		(property "Reference" "#PWR017"
+		(property "Reference" "#PWR010"
 			(at 110.49 104.14 0)
 			(effects
@@
 			(project ""
 				(path "/dc202712-23ff-46da-8ec2-2a828c683a4d/8b5991ae-ddae-4cba-9bee-b5c93b934b0b"
-					(reference "#PWR017")
+					(reference "#PWR010")
 					(unit 1)
 				)
@@
 			)
 		)
-		(property "Value" "Crystal"
+		(property "Value" "12MHz"
 			(at 214.122 102.616 90)
 			(effects
@@
 			)
 		)
-		(property "Footprint" ""
+		(property "Footprint" "Crystal:Crystal_HC49-4H_Vertical"
 			(at 210.82 101.6 0)
 			(effects
@@
 		(dnp no)
 		(fields_autoplaced yes)
-		(property "Reference" "U1"
+		(property "Reference" "U2"
 			(at 147.32 72.39 0)
 			(effects
@@
 			)
 		)
-		(property "Footprint" "DB28_TEX"
+		(property "Footprint" "Package_SO:SSOP-28_5.3x10.2mm_P0.65mm"
 			(at 114.3 82.55 0)
 			(effects
@@
 			(project ""
 				(path "/dc202712-23ff-46da-8ec2-2a828c683a4d/8b5991ae-ddae-4cba-9bee-b5c93b934b0b"
-					(reference "U1")
+					(reference "U2")
 					(unit 1)
 				)
@@
 		(dnp no)
 		(fields_autoplaced yes)
-		(property "Reference" "#PWR015"
+		(property "Reference" "#PWR012"
 			(at 194.31 116.84 0)
 			(effects
@@
 			(project "usb_microphone"
 				(path "/dc202712-23ff-46da-8ec2-2a828c683a4d/8b5991ae-ddae-4cba-9bee-b5c93b934b0b"
-					(reference "#PWR015")
+					(reference "#PWR012")
 					(unit 1)
 				)
@@
 		(on_board yes)
 		(dnp no)
-		(property "Reference" "#PWR014"
+		(property "Reference" "#PWR011"
 			(at 114.3 127 0)
 			(effects
@@
 			(project "usb_microphone"
 				(path "/dc202712-23ff-46da-8ec2-2a828c683a4d/8b5991ae-ddae-4cba-9bee-b5c93b934b0b"
-					(reference "#PWR014")
+					(reference "#PWR011")
 					(unit 1)
 				)
@@
 		(on_board yes)
 		(dnp no)
-		(property "Reference" "#PWR016"
+		(property "Reference" "#PWR06"
 			(at 76.2 91.44 0)
 			(effects
@@
 			(project ""
 				(path "/dc202712-23ff-46da-8ec2-2a828c683a4d/8b5991ae-ddae-4cba-9bee-b5c93b934b0b"
-					(reference "#PWR016")
+					(reference "#PWR06")
 					(unit 1)
 				)
@@
 		(on_board yes)
 		(dnp no)
-		(property "Reference" "C3"
+		(property "Reference" "C7"
 			(at 95.758 109.22 90)
 			(effects
@@
 			)
 		)
-		(property "Footprint" ""
+		(property "Footprint" "Capacitor_SMD:C_0603_1608Metric_Pad1.08x0.95mm_HandSolder"
 			(at 100.33 107.95 0)
 			(effects
@@
 			(project ""
 				(path "/dc202712-23ff-46da-8ec2-2a828c683a4d/8b5991ae-ddae-4cba-9bee-b5c93b934b0b"
-					(reference "C3")
+					(reference "C7")
 					(unit 1)
 				)
@@
 		(on_board yes)
 		(dnp no)
-		(property "Reference" "C5"
+		(property "Reference" "C8"
 			(at 117.094 117.094 0)
 			(effects
@@
 			)
 		)
-		(property "Footprint" ""
+		(property "Footprint" "Capacitor_SMD:C_0603_1608Metric_Pad1.08x0.95mm_HandSolder"
 			(at 114.3 118.11 0)
 			(effects
@@
 			(project ""
 				(path "/dc202712-23ff-46da-8ec2-2a828c683a4d/8b5991ae-ddae-4cba-9bee-b5c93b934b0b"
-					(reference "C5")
+					(reference "C8")
 					(unit 1)
 				)
@@
 			)
 		)
-		(property "Footprint" ""
+		(property "Footprint" "Resistor_SMD:R_0603_1608Metric_Pad0.98x0.95mm_HandSolder"
 			(at 97.79 83.312 90)
 			(effects
@@
 		(on_board yes)
 		(dnp no)
-		(property "Reference" "R9"
+		(property "Reference" "R7"
 			(at 198.628 76.2 0)
 			(effects
@@
 			)
 		)
-		(property "Footprint" ""
+		(property "Footprint" "Resistor_SMD:R_0603_1608Metric_Pad0.98x0.95mm_HandSolder"
 			(at 196.088 77.47 90)
 			(effects
@@
 			(project "usb_microphone"
 				(path "/dc202712-23ff-46da-8ec2-2a828c683a4d/8b5991ae-ddae-4cba-9bee-b5c93b934b0b"
-					(reference "R9")
+					(reference "R7")
 					(unit 1)
 				)
@@
 		(on_board yes)
 		(dnp no)
-		(property "Reference" "C15"
+		(property "Reference" "C14"
 			(at 204.47 109.474 90)
 			(effects
@@
 			)
 		)
-		(property "Footprint" ""
+		(property "Footprint" "Capacitor_SMD:C_0603_1608Metric_Pad1.08x0.95mm_HandSolder"
 			(at 208.28 104.4448 0)
 			(effects
@@
 			(project "usb_microphone"
 				(path "/dc202712-23ff-46da-8ec2-2a828c683a4d/8b5991ae-ddae-4cba-9bee-b5c93b934b0b"
-					(reference "C15")
+					(reference "C14")
 					(unit 1)
 				)
@@
 			)
 		)
-		(property "Footprint" ""
+		(property "Footprint" "Capacitor_SMD:C_0603_1608Metric_Pad1.08x0.95mm_HandSolder"
 			(at 190.5 104.4448 0)
 			(effects
@@
 		(on_board yes)
 		(dnp no)
-		(property "Reference" "R10"
+		(property "Reference" "R8"
 			(at 227.584 100.33 0)
 			(effects
@@
 			)
 		)
-		(property "Footprint" ""
+		(property "Footprint" "Resistor_SMD:R_0603_1608Metric_Pad0.98x0.95mm_HandSolder"
 			(at 224.028 101.6 90)
 			(effects
@@
 			(project "usb_microphone"
 				(path "/dc202712-23ff-46da-8ec2-2a828c683a4d/8b5991ae-ddae-4cba-9bee-b5c93b934b0b"
-					(reference "R10")
+					(reference "R8")
 					(unit 1)
 				)
@@
 		(on_board yes)
 		(dnp no)
-		(property "Reference" "#PWR013"
+		(property "Reference" "#PWR09"
 			(at 105.41 113.03 0)
 			(effects
@@
 			(project "usb_microphone"
 				(path "/dc202712-23ff-46da-8ec2-2a828c683a4d/8b5991ae-ddae-4cba-9bee-b5c93b934b0b"
-					(reference "#PWR013")
+					(reference "#PWR09")
 					(unit 1)
 				)
@@
 			)
 		)
-		(property "Footprint" ""
+		(property "Footprint" "Capacitor_SMD:C_0603_1608Metric_Pad1.08x0.95mm_HandSolder"
 			(at 190.5 94.2848 0)
 			(effects
@@
 			)
 		)
-		(property "Footprint" ""
+		(property "Footprint" "Capacitor_SMD:C_0603_1608Metric_Pad1.08x0.95mm_HandSolder"
 			(at 195.2752 93.98 0)
 			(effects
@@
 			)
 		)
-		(property "Footprint" ""
+		(property "Footprint" "Capacitor_SMD:C_0603_1608Metric_Pad1.08x0.95mm_HandSolder"
 			(at 190.5 109.5248 0)
 			(effects
@@
 		(dnp no)
 		(fields_autoplaced yes)
-		(property "Reference" "#PWR019"
+		(property "Reference" "#PWR013"
 			(at 204.47 88.9 0)
 			(effects
@@
 			(project ""
 				(path "/dc202712-23ff-46da-8ec2-2a828c683a4d/8b5991ae-ddae-4cba-9bee-b5c93b934b0b"
-					(reference "#PWR019")
+					(reference "#PWR013")
 					(unit 1)
 				)
@@
 		(on_board yes)
 		(dnp no)
-		(property "Reference" "C1"
+		(property "Reference" "C6"
 			(at 91.44 116.586 90)
 			(effects
@@
 			)
 		)
-		(property "Footprint" ""
+		(property "Footprint" "Capacitor_SMD:C_0603_1608Metric_Pad1.08x0.95mm_HandSolder"
 			(at 87.63 113.9952 0)
 			(effects
@@
 			(project "usb_microphone"
 				(path "/dc202712-23ff-46da-8ec2-2a828c683a4d/8b5991ae-ddae-4cba-9bee-b5c93b934b0b"
-					(reference "C1")
-					(unit 1)
-				)
+					(reference "C6")
+					(unit 1)
+				)

Commit message: Update Footprints for C with `10uf`
Parts:
- C7, C8: footprint Capacitor_SMD:C_0603_1608Metric_Pad1.08x0.95mm_HandSolder -> Capacitor_Tantalum_SMD:CP_EIA-3216-10_Kemet-I_HandSolder
Changed lines of the file:
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@@
 			)
 		)
-		(property "Footprint" "Capacitor_SMD:C_0603_1608Metric_Pad1.08x0.95mm_HandSolder"
+		(property "Footprint" "Capacitor_Tantalum_SMD:CP_EIA-3216-10_Kemet-I_HandSolder"
 			(at 100.33 107.95 0)
 			(effects
@@
 			)
 		)
-		(property "Footprint" "Capacitor_SMD:C_0603_1608Metric_Pad1.08x0.95mm_HandSolder"
+		(property "Footprint" "Capacitor_Tantalum_SMD:CP_EIA-3216-10_Kemet-I_HandSolder"
 			(at 114.3 118.11 0)
 			(effects
